File: kaboardv3-hw/kaboardv3-hw.kicad_sch (KiCad schematic)
At the start: 0 parts

Commit message: capture validated keyboard electrical baseline
Parts:
- added C1, C36: 1u BQ IN, Capacitor_SMD:C_0402_1005Metric, symbol Device:C
- added C10, C45, C75: 100n nRF VBUS, Capacitor_SMD:C_0402_1005Metric, symbol Device:C
- added C11, C46, C76: 12p NRF XL1, Capacitor_SMD:C_0402_1005Metric, symbol Device:C
- added C12, C47, C77: 12p NRF XL2, Capacitor_SMD:C_0402_1005Metric, symbol Device:C
- added C13, C48: 10u RGB IN, Capacitor_SMD:C_0402_1005Metric, symbol Device:C
- added C14, C49: 47u LED 5V, Capacitor_SMD:C_0402_1005Metric, symbol Device:C
- added C15, C50: 100n LED bulk, Capacitor_SMD:C_0402_1005Metric, symbol Device:C
- added C16, C51, C78: 1u OLED VCC, Capacitor_SMD:C_0402_1005Metric, symbol Device:C
- added C17, C52, C79: 100n OLED VCC, Capacitor_SMD:C_0402_1005Metric, symbol Device:C
- added C18: 100n TMAG A01, Capacitor_SMD:C_0402_1005Metric, symbol Device:C
- added C19: 100n TMAG A02, Capacitor_SMD:C_0402_1005Metric, symbol Device:C
- added C2, C37: 10u SYS, Capacitor_SMD:C_0402_1005Metric, symbol Device:C
- added C20: 100n TMAG A03, Capacitor_SMD:C_0402_1005Metric, symbol Device:C
- added C21: 100n TMAG A04, Capacitor_SMD:C_0402_1005Metric, symbol Device:C
- added C22: 100n TMAG A05, Capacitor_SMD:C_0402_1005Metric, symbol Device:C
- added C23: 100n TMAG A06, Capacitor_SMD:C_0402_1005Metric, symbol Device:C
- added C24: 100n TMAG A07, Capacitor_SMD:C_0402_1005Metric, symbol Device:C
- added C25: 100n TMAG A08, Capacitor_SMD:C_0402_1005Metric, symbol Device:C
- added C26: 100n TMAG A09, Capacitor_SMD:C_0402_1005Metric, symbol Device:C
- added C27: 100n TMAG A10, Capacitor_SMD:C_0402_1005Metric, symbol Device:C
- added C28: 100n TMAG A11, Capacitor_SMD:C_0402_1005Metric, symbol Device:C
- added C29: 100n TMAG A12, Capacitor_SMD:C_0402_1005Metric, symbol Device:C
- added C3, C38: 1u BAT, Capacitor_SMD:C_0402_1005Metric, symbol Device:C
- added C30: 100n TMAG A13, Capacitor_SMD:C_0402_1005Metric, symbol Device:C
- added C31: 100n TMAG A14, Capacitor_SMD:C_0402_1005Metric, symbol Device:C
- added C32: 100n TMAG A15, Capacitor_SMD:C_0402_1005Metric, symbol Device:C
- added C33: 100n TMAG A16, Capacitor_SMD:C_0402_1005Metric, symbol Device:C
- added C34: 100n TMAG A17, Capacitor_SMD:C_0402_1005Metric, symbol Device:C
- added C35: 100n TMAG A18, Capacitor_SMD:C_0402_1005Metric, symbol Device:C
- added C39, C4: 10u TPS IN, Capacitor_SMD:C_0402_1005Metric, symbol Device:C
- added C40, C5: 10u 3V3, Capacitor_SMD:C_0402_1005Metric, symbol Device:C
- added C41, C6: 100n STM VDD, Capacitor_SMD:C_0402_1005Metric, symbol Device:C
- added C42, C7: 100n STM VDDA, Capacitor_SMD:C_0402_1005Metric, symbol Device:C
- added C43, C73, C8: 100n nRF VDD, Capacitor_SMD:C_0402_1005Metric, symbol Device:C
- added C44, C74, C9: 100n nRF VDDH, Capacitor_SMD:C_0402_1005Metric, symbol Device:C
- added C53: 100n TMAG B01, Capacitor_SMD:C_0402_1005Metric, symbol Device:C
- added C54: 100n TMAG B02, Capacitor_SMD:C_0402_1005Metric, symbol Device:C
- added C55: 100n TMAG B03, Capacitor_SMD:C_0402_1005Metric, symbol Device:C
- added C56: 100n TMAG B04, Capacitor_SMD:C_0402_1005Metric, symbol Device:C
- added C57: 100n TMAG B05, Capacitor_SMD:C_0402_1005Metric, symbol Device:C
- added C58: 100n TMAG B06, Capacitor_SMD:C_0402_1005Metric, symbol Device:C
- added C59: 100n TMAG B07, Capacitor_SMD:C_0402_1005Metric, symbol Device:C
- added C60: 100n TMAG B08, Capacitor_SMD:C_0402_1005Metric, symbol Device:C
- added C61: 100n TMAG B09, Capacitor_SMD:C_0402_1005Metric, symbol Device:C
- added C62: 100n TMAG B10, Capacitor_SMD:C_0402_1005Metric, symbol Device:C
- added C63: 100n TMAG B11, Capacitor_SMD:C_0402_1005Metric, symbol Device:C
- added C64: 100n TMAG B12, Capacitor_SMD:C_0402_1005Metric, symbol Device:C
- added C65: 100n TMAG B13, Capacitor_SMD:C_0402_1005Metric, symbol Device:C
- added C66: 100n TMAG B14, Capacitor_SMD:C_0402_1005Metric, symbol Device:C
- added C67: 100n TMAG B15, Capacitor_SMD:C_0402_1005Metric, symbol Device:C
- added C68: 100n TMAG B16, Capacitor_SMD:C_0402_1005Metric, symbol Device:C
- added C69: 100n TMAG B17, Capacitor_SMD:C_0402_1005Metric, symbol Device:C
- added C70: 100n TMAG B18, Capacitor_SMD:C_0402_1005Metric, symbol Device:C
- added C71: 10u USB 5V IN, Capacitor_SMD:C_0402_1005Metric, symbol Device:C
- added C72: 10u RX 3V3, Capacitor_SMD:C_0402_1005Metric, symbol Device:C
- added D1, D21, D41: ESD441DPYR USB VBUS, Diode_SMD:D_0201_0603Metric, symbol kaboard_custom:ESD441DPYR_PASSIVE
- added D10, D30: WL-ICLED 1312020030000 #8, kaboard_custom:U_Wurth_WL-ICLED_1312020030000, symbol kaboard_custom:WL_ICLED_1312020030000
- added D11, D31: WL-ICLED 1312020030000 #9, kaboard_custom:U_Wurth_WL-ICLED_1312020030000, symbol kaboard_custom:WL_ICLED_1312020030000
- added D12, D32: WL-ICLED 1312020030000 #10, kaboard_custom:U_Wurth_WL-ICLED_1312020030000, symbol kaboard_custom:WL_ICLED_1312020030000
- added D13, D33: WL-ICLED 1312020030000 #11, kaboard_custom:U_Wurth_WL-ICLED_1312020030000, symbol kaboard_custom:WL_ICLED_1312020030000
- added D14, D34: WL-ICLED 1312020030000 #12, kaboard_custom:U_Wurth_WL-ICLED_1312020030000, symbol kaboard_custom:WL_ICLED_1312020030000
- added D15, D35: WL-ICLED 1312020030000 #13, kaboard_custom:U_Wurth_WL-ICLED_1312020030000, symbol kaboard_custom:WL_ICLED_1312020030000
- added D16, D36: WL-ICLED 1312020030000 #14, kaboard_custom:U_Wurth_WL-ICLED_1312020030000, symbol kaboard_custom:WL_ICLED_1312020030000
- added D17, D37: WL-ICLED 1312020030000 #15, kaboard_custom:U_Wurth_WL-ICLED_1312020030000, symbol kaboard_custom:WL_ICLED_1312020030000
- added D18, D38: WL-ICLED 1312020030000 #16, kaboard_custom:U_Wurth_WL-ICLED_1312020030000, symbol kaboard_custom:WL_ICLED_1312020030000
- added D19, D39: WL-ICLED 1312020030000 #17, kaboard_custom:U_Wurth_WL-ICLED_1312020030000, symbol kaboard_custom:WL_ICLED_1312020030000
- added D2: LEFT STATUS LED, LED_SMD:LED_0603_1608Metric, symbol Device:LED
- added D20, D40: WL-ICLED 1312020030000 #18, kaboard_custom:U_Wurth_WL-ICLED_1312020030000, symbol kaboard_custom:WL_ICLED_1312020030000
- added D22: RIGHT STATUS LED, LED_SMD:LED_0603_1608Metric, symbol Device:LED
- added D23, D3: WL-ICLED 1312020030000 #1, kaboard_custom:U_Wurth_WL-ICLED_1312020030000, symbol kaboard_custom:WL_ICLED_1312020030000
- added D24, D4: WL-ICLED 1312020030000 #2, kaboard_custom:U_Wurth_WL-ICLED_1312020030000, symbol kaboard_custom:WL_ICLED_1312020030000
- added D25, D5: WL-ICLED 1312020030000 #3, kaboard_custom:U_Wurth_WL-ICLED_1312020030000, symbol kaboard_custom:WL_ICLED_1312020030000
- added D26, D6: WL-ICLED 1312020030000 #4, kaboard_custom:U_Wurth_WL-ICLED_1312020030000, symbol kaboard_custom:WL_ICLED_1312020030000
- added D27, D7: WL-ICLED 1312020030000 #5, kaboard_custom:U_Wurth_WL-ICLED_1312020030000, symbol kaboard_custom:WL_ICLED_1312020030000
- added D28, D8: WL-ICLED 1312020030000 #6, kaboard_custom:U_Wurth_WL-ICLED_1312020030000, symbol kaboard_custom:WL_ICLED_1312020030000
- added D29, D9: WL-ICLED 1312020030000 #7, kaboard_custom:U_Wurth_WL-ICLED_1312020030000, symbol kaboard_custom:WL_ICLED_1312020030000
- added D42: STATUS LED, LED_SMD:LED_0603_1608Metric, symbol Device:LED
- added J1, J11, J6: USB_C_Receptacle_PowerOnly_6P, Connector_USB:USB_C_Receptacle_GCT_USB4125-xx-x-0190_6P_TopMnt_Horizontal, symbol Connector:USB_C_Receptacle_PowerOnly_6P
- added J10, J5: nRF SWD, Connector_PinHeader_2.54mm:PinHeader_1x05_P2.54mm_Vertical, symbol Connector_Generic:Conn_01x05
- added J12, J3, J8: SH1106 1.3in 4-wire OLED, Connector_PinHeader_2.54mm:PinHeader_1x04_P2.54mm_Vertical, symbol Connector_Generic:Conn_01x04
- added J13: Receiver nRF SWD, Connector_PinHeader_2.54mm:PinHeader_1x05_P2.54mm_Vertical, symbol Connector_Generic:Conn_01x05
- added J2, J7: AS584070 BATTERY / 10k NTC, Connector_JST:JST_PH_B3B-PH-K_1x03_P2.00mm_Vertical, symbol Connector:Conn_01x03_Pin
- added J4, J9: STM32 SWD, Connector_PinHeader_2.54mm:PinHeader_1x05_P2.54mm_Vertical, symbol Connector_Generic:Conn_01x05
- added L1, L3: 2.2uH TPS63031, Inductor_SMD:L_0603_1608Metric, symbol Device:L
- added L2, L4: 1uH RGB BOOST, Inductor_SMD:L_0603_1608Metric, symbol Device:L
- added L5, L6, L7: 10uH nRF DCDC, Inductor_SMD:L_0603_1608Metric, symbol Device:L
- added R1, R15, R29: 5.1k USB CC1, Resistor_SMD:R_0402_1005Metric, symbol Device:R
- added R10, R24: 330k BAT_SENSE bottom, Resistor_SMD:R_0402_1005Metric, symbol Device:R
- added R11, R25: 330R RGB data, Resistor_SMD:R_0402_1005Metric, symbol Device:R
- added R12, R26: 732k RGB FB top, Resistor_SMD:R_0402_1005Metric, symbol Device:R
- added R13, R27: 100k RGB FB bottom, Resistor_SMD:R_0402_1005Metric, symbol Device:R
- added R14, R28, R34: 1k STATUS LED, Resistor_SMD:R_0402_1005Metric, symbol Device:R
- added R16, R2, R30: 5.1k USB CC2, Resistor_SMD:R_0402_1005Metric, symbol Device:R
- added R17, R3: 18k BQ ILIM/VSET, Resistor_SMD:R_0402_1005Metric, symbol Device:R
- added R18, R4: 845R BQ ISET, Resistor_SMD:R_0402_1005Metric, symbol Device:R
- added R19, R31, R5: 10k nRF RESET pullup, Resistor_SMD:R_0402_1005Metric, symbol Device:R
- added R20, R6: 10k BOOT0 pulldown, Resistor_SMD:R_0402_1005Metric, symbol Device:R
- added R21, R32, R7: 4.7k I2C SDA pullup, Resistor_SMD:R_0402_1005Metric, symbol Device:R
- added R22, R33, R8: 4.7k I2C SCL pullup, Resistor_SMD:R_0402_1005Metric, symbol Device:R
- added R23, R9: 1M BAT_SENSE top, Resistor_SMD:R_0402_1005Metric, symbol Device:R
- added U1, U27: STM32G431RBTx, Package_QFP:LQFP-64_10x10mm_P0.5mm, symbol MCU_ST_STM32G4:STM32G431RBTx
- added U10: TMAG5253BA3IQDMRR A02, Package_SON:Texas_X2SON-4-1EP_1.1x1.4mm_P0.5mm_EP0.8x0.6mm, symbol kaboard_custom:TMAG5253BA3IQDMRR
- added U11: TMAG5253BA3IQDMRR A03, Package_SON:Texas_X2SON-4-1EP_1.1x1.4mm_P0.5mm_EP0.8x0.6mm, symbol kaboard_custom:TMAG5253BA3IQDMRR
- added U12: TMAG5253BA3IQDMRR A04, Package_SON:Texas_X2SON-4-1EP_1.1x1.4mm_P0.5mm_EP0.8x0.6mm, symbol kaboard_custom:TMAG5253BA3IQDMRR
- added U13: TMAG5253BA3IQDMRR A05, Package_SON:Texas_X2SON-4-1EP_1.1x1.4mm_P0.5mm_EP0.8x0.6mm, symbol kaboard_custom:TMAG5253BA3IQDMRR
- added U14: TMAG5253BA3IQDMRR A06, Package_SON:Texas_X2SON-4-1EP_1.1x1.4mm_P0.5mm_EP0.8x0.6mm, symbol kaboard_custom:TMAG5253BA3IQDMRR
- added U15: TMAG5253BA3IQDMRR A07, Package_SON:Texas_X2SON-4-1EP_1.1x1.4mm_P0.5mm_EP0.8x0.6mm, symbol kaboard_custom:TMAG5253BA3IQDMRR
- added U16: TMAG5253BA3IQDMRR A08, Package_SON:Texas_X2SON-4-1EP_1.1x1.4mm_P0.5mm_EP0.8x0.6mm, symbol kaboard_custom:TMAG5253BA3IQDMRR
- added U17: TMAG5253BA3IQDMRR A09, Package_SON:Texas_X2SON-4-1EP_1.1x1.4mm_P0.5mm_EP0.8x0.6mm, symbol kaboard_custom:TMAG5253BA3IQDMRR
- added U18: TMAG5253BA3IQDMRR A10, Package_SON:Texas_X2SON-4-1EP_1.1x1.4mm_P0.5mm_EP0.8x0.6mm, symbol kaboard_custom:TMAG5253BA3IQDMRR
- added U19: TMAG5253BA3IQDMRR A11, Package_SON:Texas_X2SON-4-1EP_1.1x1.4mm_P0.5mm_EP0.8x0.6mm, symbol kaboard_custom:TMAG5253BA3IQDMRR
- added U2, U28, U52: MDBT50Q-1MV2, RF_Module:Raytac_MDBT50Q, symbol RF_Module:MDBT50Q-1MV2
- added U20: TMAG5253BA3IQDMRR A12, Package_SON:Texas_X2SON-4-1EP_1.1x1.4mm_P0.5mm_EP0.8x0.6mm, symbol kaboard_custom:TMAG5253BA3IQDMRR
- added U21: TMAG5253BA3IQDMRR A13, Package_SON:Texas_X2SON-4-1EP_1.1x1.4mm_P0.5mm_EP0.8x0.6mm, symbol kaboard_custom:TMAG5253BA3IQDMRR
- added U22: TMAG5253BA3IQDMRR A14, Package_SON:Texas_X2SON-4-1EP_1.1x1.4mm_P0.5mm_EP0.8x0.6mm, symbol kaboard_custom:TMAG5253BA3IQDMRR
- added U23: TMAG5253BA3IQDMRR A15, Package_SON:Texas_X2SON-4-1EP_1.1x1.4mm_P0.5mm_EP0.8x0.6mm, symbol kaboard_custom:TMAG5253BA3IQDMRR
- added U24: TMAG5253BA3IQDMRR A16, Package_SON:Texas_X2SON-4-1EP_1.1x1.4mm_P0.5mm_EP0.8x0.6mm, symbol kaboard_custom:TMAG5253BA3IQDMRR
- added U25: TMAG5253BA3IQDMRR A17, Package_SON:Texas_X2SON-4-1EP_1.1x1.4mm_P0.5mm_EP0.8x0.6mm, symbol kaboard_custom:TMAG5253BA3IQDMRR
- added U26: TMAG5253BA3IQDMRR A18, Package_SON:Texas_X2SON-4-1EP_1.1x1.4mm_P0.5mm_EP0.8x0.6mm, symbol kaboard_custom:TMAG5253BA3IQDMRR
- added U29, U3: BQ25185DLHR, Package_DFN_QFN:Texas_DLH0010A_WSON-10-1EP_2.2x2mm_P0.4mm_EP0.9x1.5mm, symbol kaboard_custom:BQ25185DLHR
- added U30, U4: TPS63031DSK, Package_SON:WSON-10-1EP_2.5x2.5mm_P0.5mm_EP1.2x2mm, symbol Regulator_Switching:TPS63031DSK
- added U31, U5: TPS61022 RGB BOOST, Package_DFN_QFN:Texas_RWU0007A_VQFN-7_2x2mm_P0.5mm, symbol Converter_DCDC:TPS61022
- added U32, U6: 74AHCT1G125, Package_TO_SOT_SMD:SOT-23-5, symbol 74xGxx:74AHCT1G125
- added U33, U54, U7: TPS22919DCK, Package_TO_SOT_SMD:SOT-363_SC-70-6, symbol Power_Management:TPS22919DCK
- added U34: TMAG5253BA3IQDMRR B01, Package_SON:Texas_X2SON-4-1EP_1.1x1.4mm_P0.5mm_EP0.8x0.6mm, symbol kaboard_custom:TMAG5253BA3IQDMRR
- added U35: TMAG5253BA3IQDMRR B02, Package_SON:Texas_X2SON-4-1EP_1.1x1.4mm_P0.5mm_EP0.8x0.6mm, symbol kaboard_custom:TMAG5253BA3IQDMRR
- added U36: TMAG5253BA3IQDMRR B03, Package_SON:Texas_X2SON-4-1EP_1.1x1.4mm_P0.5mm_EP0.8x0.6mm, symbol kaboard_custom:TMAG5253BA3IQDMRR
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Connections:
- new net L_3V3: C10.1, C13.1, C18.1, C19.1, C20.1, C21.1, C22.1, C23.1, C24.1, C25.1, C26.1, C27.1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
- new net L_BAT: C3.1, J2.1 (Pin_1), R9.1, U3.2 (BAT)
- new net L_BAT_SENSE: R10.1, R9.2, U2.10 (P0.29)
- new net L_BOOT0: R6.1, U1.61 (PB8)
- new net L_BQ_ILIM: R3.1, U3.7 (ILIM/VSET)
- new net L_BQ_ISET: R4.1, U3.8 (ISET)
- new net L_DISPLAY_EN: U2.49 (P0.25), U7.3 (ON)
- new net L_DISPLAY_SCL: J3.3 (Pin_3), R8.2, U2.19 (P0.26)
- new net L_DISPLAY_SDA: J3.4 (Pin_4), R7.2, U2.16 (P0.27)
- new net L_GND: C1.2, C10.2, C11.2, C12.2, C13.2, C14.2, C15.2, C16.2, C17.2, C18.2, C19.2, C2.2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
- new net L_HALL_EN_A: U1.38 (PC6), U10.3 (EN), U11.3 (EN), U12.3 (EN), U13.3 (EN), U14.3 (EN), U9.3 (EN)
- new net L_HALL_EN_B: U1.39 (PC7), U15.3 (EN), U16.3 (EN), U17.3 (EN), U18.3 (EN), U19.3 (EN), U20.3 (EN)
- new net L_HALL_EN_C: U1.40 (PC8), U21.3 (EN), U22.3 (EN), U23.3 (EN), U24.3 (EN), U25.3 (EN), U26.3 (EN)
- new net L_HALL_OUT_01: U1.8 (PC0), U9.4 (OUT)
- new net L_HALL_OUT_02: U1.9 (PC1), U10.4 (OUT)
- new net L_HALL_OUT_03: U1.10 (PC2), U11.4 (OUT)
- new net L_HALL_OUT_04: U1.11 (PC3), U12.4 (OUT)
- new net L_HALL_OUT_05: U1.12 (PA0), U13.4 (OUT)
- new net L_HALL_OUT_06: U1.13 (PA1), U14.4 (OUT)
- new net L_HALL_OUT_07: U1.14 (PA2), U15.4 (OUT)
- new net L_HALL_OUT_08: U1.17 (PA3), U16.4 (OUT)
- new net L_HALL_OUT_09: U1.18 (PA4), U17.4 (OUT)
- new net L_HALL_OUT_10: U1.19 (PA5), U18.4 (OUT)
- new net L_HALL_OUT_11: U1.20 (PA6), U19.4 (OUT)
- new net L_HALL_OUT_12: U1.21 (PA7), U20.4 (OUT)
- new net L_HALL_OUT_13: U1.22 (PC4), U21.4 (OUT)
- new net L_HALL_OUT_14: U1.23 (PC5), U22.4 (OUT)
- new net L_HALL_OUT_15: U1.24 (PB0), U23.4 (OUT)
- new net L_HALL_OUT_16: U1.25 (PB1), U24.4 (OUT)
- new net L_HALL_OUT_17: U1.26 (PB2), U25.4 (OUT)
- new net L_HALL_OUT_18: U1.33 (PB11), U26.4 (OUT)
- new net L_LED_5V: C14.1, C15.1, D10.1 (VDD), D11.1 (VDD), D12.1 (VDD), D13.1 (VDD), D14.1 (VDD), D15.1 (VDD), D16.1 (VDD), D17.1 (VDD), D18.1 (VDD), D19.1 (VDD)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
- new net L_NRF_DCCH: L6.1, U2.31 (DCCH)
- new net L_NRF_RESET_N: J5.5 (Pin_5), R5.1, U2.40 (P0.18)
- new net L_NRF_XL1: C11.1, U2.17 (P0.00), Y1.1
- new net L_NRF_XL2: C12.1, U2.18 (P0.01), Y1.2
- new net L_NTC: J2.2 (Pin_2), U3.6 (TS/MR)
- new net L_OLED_VCC: C16.1, C17.1, J3.1 (Pin_1), U7.6 (OUT)
- new net L_RGB_DATA_3V3: U1.42 (PA8), U6.2
- new net L_RGB_DATA_5V: R11.1, U6.4
- new net L_RGB_DIN_01: D3.2 (DIN), R11.2
- new net L_RGB_DIN_02: D3.3 (DOUT), D4.2 (DIN)
- new net L_RGB_DIN_03: D4.3 (DOUT), D5.2 (DIN)
- new net L_RGB_DIN_04: D5.3 (DOUT), D6.2 (DIN)
- new net L_RGB_DIN_05: D6.3 (DOUT), D7.2 (DIN)
- new net L_RGB_DIN_06: D7.3 (DOUT), D8.2 (DIN)
- new net L_RGB_DIN_07: D8.3 (DOUT), D9.2 (DIN)
- new net L_RGB_DIN_08: D10.2 (DIN), D9.3 (DOUT)
- new net L_RGB_DIN_09: D10.3 (DOUT), D11.2 (DIN)
- new net L_RGB_DIN_10: D11.3 (DOUT), D12.2 (DIN)
- new net L_RGB_DIN_11: D12.3 (DOUT), D13.2 (DIN)
- new net L_RGB_DIN_12: D13.3 (DOUT), D14.2 (DIN)
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
Commit message: organize schematic into readable functional sections
Parts:
- D10: value WL-ICLED 1312020030000 #8 -> WL-ICLED A08
- D11: value WL-ICLED 1312020030000 #9 -> WL-ICLED A09
- D12: value WL-ICLED 1312020030000 #10 -> WL-ICLED A10
- D13: value WL-ICLED 1312020030000 #11 -> WL-ICLED A11
- D14: value WL-ICLED 1312020030000 #12 -> WL-ICLED A12
- D15: value WL-ICLED 1312020030000 #13 -> WL-ICLED A13
- D16: value WL-ICLED 1312020030000 #14 -> WL-ICLED A14
- D17: value WL-ICLED 1312020030000 #15 -> WL-ICLED A15
- D18: value WL-ICLED 1312020030000 #16 -> WL-ICLED A16
- D19: value WL-ICLED 1312020030000 #17 -> WL-ICLED A17
- D20: value WL-ICLED 1312020030000 #18 -> WL-ICLED A18
- D23: value WL-ICLED 1312020030000 #1 -> WL-ICLED B01
- D24: value WL-ICLED 1312020030000 #2 -> WL-ICLED B02
- D25: value WL-ICLED 1312020030000 #3 -> WL-ICLED B03
- D26: value WL-ICLED 1312020030000 #4 -> WL-ICLED B04
- D27: value WL-ICLED 1312020030000 #5 -> WL-ICLED B05
- D28: value WL-ICLED 1312020030000 #6 -> WL-ICLED B06
- D29: value WL-ICLED 1312020030000 #7 -> WL-ICLED B07
- D3: value WL-ICLED 1312020030000 #1 -> WL-ICLED A01
- D30: value WL-ICLED 1312020030000 #8 -> WL-ICLED B08
- D31: value WL-ICLED 1312020030000 #9 -> WL-ICLED B09
- D32: value WL-ICLED 1312020030000 #10 -> WL-ICLED B10
- D33: value WL-ICLED 1312020030000 #11 -> WL-ICLED B11
- D34: value WL-ICLED 1312020030000 #12 -> WL-ICLED B12
- D35: value WL-ICLED 1312020030000 #13 -> WL-ICLED B13
- D36: value WL-ICLED 1312020030000 #14 -> WL-ICLED B14
- D37: value WL-ICLED 1312020030000 #15 -> WL-ICLED B15
- D38: value WL-ICLED 1312020030000 #16 -> WL-ICLED B16
- D39: value WL-ICLED 1312020030000 #17 -> WL-ICLED B17
- D4: value WL-ICLED 1312020030000 #2 -> WL-ICLED A02
- D40: value WL-ICLED 1312020030000 #18 -> WL-ICLED B18
- D5: value WL-ICLED 1312020030000 #3 -> WL-ICLED A03
- D6: value WL-ICLED 1312020030000 #4 -> WL-ICLED A04
- D7: value WL-ICLED 1312020030000 #5 -> WL-ICLED A05
- D8: value WL-ICLED 1312020030000 #6 -> WL-ICLED A06
- D9: value WL-ICLED 1312020030000 #7 -> WL-ICLED A07
- U10: value TMAG5253BA3IQDMRR A02 -> TMAG5253 A02
- U11: value TMAG5253BA3IQDMRR A03 -> TMAG5253 A03
- U12: value TMAG5253BA3IQDMRR A04 -> TMAG5253 A04
- U13: value TMAG5253BA3IQDMRR A05 -> TMAG5253 A05
- U14: value TMAG5253BA3IQDMRR A06 -> TMAG5253 A06
- U15: value TMAG5253BA3IQDMRR A07 -> TMAG5253 A07
- U16: value TMAG5253BA3IQDMRR A08 -> TMAG5253 A08
- U17: value TMAG5253BA3IQDMRR A09 -> TMAG5253 A09
- U18: value TMAG5253BA3IQDMRR A10 -> TMAG5253 A10
- U19: value TMAG5253BA3IQDMRR A11 -> TMAG5253 A11
- U20: value TMAG5253BA3IQDMRR A12 -> TMAG5253 A12
- U21: value TMAG5253BA3IQDMRR A13 -> TMAG5253 A13
- U22: value TMAG5253BA3IQDMRR A14 -> TMAG5253 A14
- U23: value TMAG5253BA3IQDMRR A15 -> TMAG5253 A15
- U24: value TMAG5253BA3IQDMRR A16 -> TMAG5253 A16
- U25: value TMAG5253BA3IQDMRR A17 -> TMAG5253 A17
- U26: value TMAG5253BA3IQDMRR A18 -> TMAG5253 A18
- U34: value TMAG5253BA3IQDMRR B01 -> TMAG5253 B01
- U35: value TMAG5253BA3IQDMRR B02 -> TMAG5253 B02
- U36: value TMAG5253BA3IQDMRR B03 -> TMAG5253 B03
- U37: value TMAG5253BA3IQDMRR B04 -> TMAG5253 B04
- U38: value TMAG5253BA3IQDMRR B05 -> TMAG5253 B05
- U39: value TMAG5253BA3IQDMRR B06 -> TMAG5253 B06
- U40: value TMAG5253BA3IQDMRR B07 -> TMAG5253 B07
- U41: value TMAG5253BA3IQDMRR B08 -> TMAG5253 B08
- U42: value TMAG5253BA3IQDMRR B09 -> TMAG5253 B09
- U43: value TMAG5253BA3IQDMRR B10 -> TMAG5253 B10
- U44: value TMAG5253BA3IQDMRR B11 -> TMAG5253 B11
- U45: value TMAG5253BA3IQDMRR B12 -> TMAG5253 B12
- U46: value TMAG5253BA3IQDMRR B13 -> TMAG5253 B13
- U47: value TMAG5253BA3IQDMRR B14 -> TMAG5253 B14
- U48: value TMAG5253BA3IQDMRR B15 -> TMAG5253 B15
- U49: value TMAG5253BA3IQDMRR B16 -> TMAG5253 B16
- U50: value TMAG5253BA3IQDMRR B17 -> TMAG5253 B17
- U51: value TMAG5253BA3IQDMRR B18 -> TMAG5253 B18
- U9: value TMAG5253BA3IQDMRR A01 -> TMAG5253 A01
Other:
- note added: "18× TMAG5253 — 3 ENABLE GROUPS / 18 ADC CHANNELS"
- note added: "18× WL-ICLED — 5V SWITCHED RAIL / AHCT DATA LEVEL SHIFT"
- note added: "DISPLAY: 4-WIRE SH1106 MODULE (VCC / GND / SCL / SDA)"
- note added: "KABOARD V3 — ELECTRICAL SCHEMATIC"
- note added: "LEFT HALF — INDEPENDENT 1S LiPo / WIRELESS"
- note added: "L_* = LEFT HALF R_* = RIGHT HALF RX_* = USB RECEIVER"
- note added: "OPTIONAL DISPLAY: 4-WIRE SH1106 MODULE"
- note added: "POWER / CHARGE / 3V3 / 5V RGB"
- note added: "RECEIVER — USB HID / nRF52840"
- note added: "RIGHT HALF — INDEPENDENT 1S LiPo / WIRELESS"
- note added: "STM32 ACQUISITION / CALIBRATION / ACTUATION"
- note added: "SWD: STM32 + nRF52840"
- note added: "SWD: nRF52840"
- note added: "USB POWER / 3V3 / DISPLAY"
- note added: "nRF52840 RADIO / BATTERY TELEMETRY / I²C"

Commit message: wire local schematic blocks for readability
Connections:
- net L_LED_5V: now also U5.4 (FB)
- net L_RGB_FB: no longer U5.4 (FB)
- net R_LED_5V: now also U31.4 (FB)
- net R_RGB_FB: no longer U31.4 (FB)
- net L_RGB_DIN_02: no longer names the net of D3.3 (DOUT), D4.2 (DIN)
- net L_RGB_DIN_03: no longer names the net of D4.3 (DOUT), D5.2 (DIN)
- net L_RGB_DIN_04: no longer names the net of D5.3 (DOUT), D6.2 (DIN)
- net L_RGB_DIN_05: no longer names the net of D6.3 (DOUT), D7.2 (DIN)
- net L_RGB_DIN_06: no longer names the net of D7.3 (DOUT), D8.2 (DIN)
- net L_RGB_DIN_08: no longer names the net of D10.2 (DIN), D9.3 (DOUT)
- net L_RGB_DIN_09: no longer names the net of D10.3 (DOUT), D11.2 (DIN)
- net L_RGB_DIN_10: no longer names the net of D11.3 (DOUT), D12.2 (DIN)
- net L_RGB_DIN_11: no longer names the net of D12.3 (DOUT), D13.2 (DIN)
- net L_RGB_DIN_12: no longer names the net of D13.3 (DOUT), D14.2 (DIN)
- net L_RGB_DIN_14: no longer names the net of D15.3 (DOUT), D16.2 (DIN)
- net L_RGB_DIN_15: no longer names the net of D16.3 (DOUT), D17.2 (DIN)
- net L_RGB_DIN_16: no longer names the net of D17.3 (DOUT), D18.2 (DIN)
- net L_RGB_DIN_17: no longer names the net of D18.3 (DOUT), D19.2 (DIN)
- net L_RGB_DIN_18: no longer names the net of D19.3 (DOUT), D20.2 (DIN)
- net R_RGB_DIN_02: no longer names the net of D23.3 (DOUT), D24.2 (DIN)
- net R_RGB_DIN_03: no longer names the net of D24.3 (DOUT), D25.2 (DIN)
- net R_RGB_DIN_04: no longer names the net of D25.3 (DOUT), D26.2 (DIN)
- net R_RGB_DIN_05: no longer names the net of D26.3 (DOUT), D27.2 (DIN)
- net R_RGB_DIN_06: no longer names the net of D27.3 (DOUT), D28.2 (DIN)
- net R_RGB_DIN_08: no longer names the net of D29.3 (DOUT), D30.2 (DIN)
- net R_RGB_DIN_09: no longer names the net of D30.3 (DOUT), D31.2 (DIN)
- net R_RGB_DIN_10: no longer names the net of D31.3 (DOUT), D32.2 (DIN)
- net R_RGB_DIN_11: no longer names the net of D32.3 (DOUT), D33.2 (DIN)
- net R_RGB_DIN_12: no longer names the net of D33.3 (DOUT), D34.2 (DIN)
- net R_RGB_DIN_14: no longer names the net of D35.3 (DOUT), D36.2 (DIN)
- net R_RGB_DIN_15: no longer names the net of D36.3 (DOUT), D37.2 (DIN)
- net R_RGB_DIN_16: no longer names the net of D37.3 (DOUT), D38.2 (DIN)
- net R_RGB_DIN_17: no longer names the net of D38.3 (DOUT), D39.2 (DIN)
- net R_RGB_DIN_18: no longer names the net of D39.3 (DOUT), D40.2 (DIN)
- no-connect marks 162 -> 164

Commit message: wire receiver OLED power path
Connections:
- net RX_OLED_VCC: no longer J12.1 (Pin_1), U54.6 (OUT)
- new net: J12.1 (Pin_1), U54.6 (OUT)
Changed lines of the file:
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@@
 		)
 	)
+	(wire
+		(pts
+			(xy 1009.65 217.17)
+			(xy 1019.81 217.17)
+		)
+	)
+	(wire
+		(pts
+			(xy 1019.81 217.17)
+			(xy 1019.81 267.97)
+		)
+	)
+	(wire
+		(pts
+			(xy 1019.81 267.97)
+			(xy 994.41 267.97)
+		)
+	)
+	(wire
+		(pts
+			(xy 999.49 227.33)
+			(xy 1024.89 227.33)
+		)
+	)
+	(wire
+		(pts
+			(xy 1024.89 227.33)
+			(xy 1024.89 270.51)
+		)
+	)
+	(wire
+		(pts
+			(xy 1024.89 270.51)
+			(xy 994.41 270.51)
+		)
+	)
 	(text "KABOARD V3 — ELECTRICAL SCHEMATIC"
 		(at 530 35 0)
@@
 	)
 	(label "RX_GND"
-		(at 999.49 227.33 0)
-		(effects
-			(font
-				(size 1.27 1.27)
-			)
-			(justify left bottom)
-		)
-	)
-	(label "RX_GND"
 		(at 869.95 435.61 0)
 		(effects
@@
 	)
 	(label "RX_OLED_VCC"
-		(at 1009.65 217.17 0)
-		(effects
-			(font
-				(size 1.27 1.27)
-			)
-			(justify left bottom)
-		)
-	)
-	(label "RX_OLED_VCC"
-		(at 994.41 267.97 180)
-		(effects
-			(font
-				(size 1.27 1.27)
-			)
-			(justify right bottom)
-		)
-	)
-	(label "RX_OLED_VCC"
 		(at 985.52 231.14 0)
 		(effects
@@
 		)
 	)
-	(label "RX_GND"
-		(at 994.41 270.51 180)
-		(effects
-			(font
-				(size 1.27 1.27)
-			)
-			(justify right bottom)
-		)
-	)
 	(label "L_USB_VBUS"
 		(at 49.53 160.02 0)
@@
 		(effects
 			(font
+				(size 1.27 1.27)
+			)
+			(justify left bottom)
+		)
+	)
+	(label "RX_GND"
+		(at 1024.89 270.51 0)
+		(effects
+			(font

Commit message: Finalize split board layout and documentation
Parts:
- U10, U11, U12, U13, U14, U15, U16, U17, U18, U19, U20, U21, U22, U23, U24, U25, U26, U34, U35, U36, U37, U38, U39, U40, U41, U42, U43, U44, U45, U46, U47, U48, U49, U50, U51, U9: footprint Package_SON:Texas_X2SON-4-1EP_1.1x1.4mm_P0.5mm_EP0.8x0.6mm -> kaboard_custom:Kaboard_JadePro_TMAG5253
Connections:
- no-connect marks 164 -> 162

Commit message: organize unified schematics
Parts:
- removed C1, C36: 1u BQ IN, Capacitor_SMD:C_0402_1005Metric, symbol Device:C
- removed C10, C45, C75: 100n nRF VBUS, Capacitor_SMD:C_0402_1005Metric, symbol Device:C
- removed C11, C46, C76: 12p NRF XL1, Capacitor_SMD:C_0402_1005Metric, symbol Device:C
- removed C12, C47, C77: 12p NRF XL2, Capacitor_SMD:C_0402_1005Metric, symbol Device:C
- removed C13, C48: 10u RGB IN, Capacitor_SMD:C_0402_1005Metric, symbol Device:C
- removed C14, C49: 47u LED 5V, Capacitor_SMD:C_0402_1005Metric, symbol Device:C
- removed C15, C50: 100n LED bulk, Capacitor_SMD:C_0402_1005Metric, symbol Device:C
- removed C16, C51, C78: 1u OLED VCC, Capacitor_SMD:C_0402_1005Metric, symbol Device:C
- removed C17, C52, C79: 100n OLED VCC, Capacitor_SMD:C_0402_1005Metric, symbol Device:C
- removed C18: 100n TMAG A01, Capacitor_SMD:C_0402_1005Metric, symbol Device:C
- removed C19: 100n TMAG A02, Capacitor_SMD:C_0402_1005Metric, symbol Device:C
- removed C2, C37: 10u SYS, Capacitor_SMD:C_0402_1005Metric, symbol Device:C
- removed C20: 100n TMAG A03, Capacitor_SMD:C_0402_1005Metric, symbol Device:C
- removed C21: 100n TMAG A04, Capacitor_SMD:C_0402_1005Metric, symbol Device:C
- removed C22: 100n TMAG A05, Capacitor_SMD:C_0402_1005Metric, symbol Device:C
- removed C23: 100n TMAG A06, Capacitor_SMD:C_0402_1005Metric, symbol Device:C
- removed C24: 100n TMAG A07, Capacitor_SMD:C_0402_1005Metric, symbol Device:C
- removed C25: 100n TMAG A08, Capacitor_SMD:C_0402_1005Metric, symbol Device:C
- removed C26: 100n TMAG A09, Capacitor_SMD:C_0402_1005Metric, symbol Device:C
- removed C27: 100n TMAG A10, Capacitor_SMD:C_0402_1005Metric, symbol Device:C
- removed C28: 100n TMAG A11, Capacitor_SMD:C_0402_1005Metric, symbol Device:C
- removed C29: 100n TMAG A12, Capacitor_SMD:C_0402_1005Metric, symbol Device:C
- removed C3, C38: 1u BAT, Capacitor_SMD:C_0402_1005Metric, symbol Device:C
- removed C30: 100n TMAG A13, Capacitor_SMD:C_0402_1005Metric, symbol Device:C
- removed C31: 100n TMAG A14, Capacitor_SMD:C_0402_1005Metric, symbol Device:C
- removed C32: 100n TMAG A15, Capacitor_SMD:C_0402_1005Metric, symbol Device:C
- removed C33: 100n TMAG A16, Capacitor_SMD:C_0402_1005Metric, symbol Device:C
- removed C34: 100n TMAG A17, Capacitor_SMD:C_0402_1005Metric, symbol Device:C
- removed C35: 100n TMAG A18, Capacitor_SMD:C_0402_1005Metric, symbol Device:C
- removed C39, C4: 10u TPS IN, Capacitor_SMD:C_0402_1005Metric, symbol Device:C
- removed C40, C5: 10u 3V3, Capacitor_SMD:C_0402_1005Metric, symbol Device:C
- removed C41, C6: 100n STM VDD, Capacitor_SMD:C_0402_1005Metric, symbol Device:C
- removed C42, C7: 100n STM VDDA, Capacitor_SMD:C_0402_1005Metric, symbol Device:C
- removed C43, C73, C8: 100n nRF VDD, Capacitor_SMD:C_0402_1005Metric, symbol Device:C
- removed C44, C74, C9: 100n nRF VDDH, Capacitor_SMD:C_0402_1005Metric, symbol Device:C
- removed C53: 100n TMAG B01, Capacitor_SMD:C_0402_1005Metric, symbol Device:C
- removed C54: 100n TMAG B02, Capacitor_SMD:C_0402_1005Metric, symbol Device:C
- removed C55: 100n TMAG B03, Capacitor_SMD:C_0402_1005Metric, symbol Device:C
- removed C56: 100n TMAG B04, Capacitor_SMD:C_0402_1005Metric, symbol Device:C
- removed C57: 100n TMAG B05, Capacitor_SMD:C_0402_1005Metric, symbol Device:C
- removed C58: 100n TMAG B06, Capacitor_SMD:C_0402_1005Metric, symbol Device:C
- removed C59: 100n TMAG B07, Capacitor_SMD:C_0402_1005Metric, symbol Device:C
- removed C60: 100n TMAG B08, Capacitor_SMD:C_0402_1005Metric, symbol Device:C
- removed C61: 100n TMAG B09, Capacitor_SMD:C_0402_1005Metric, symbol Device:C
- removed C62: 100n TMAG B10, Capacitor_SMD:C_0402_1005Metric, symbol Device:C
- removed C63: 100n TMAG B11, Capacitor_SMD:C_0402_1005Metric, symbol Device:C
- removed C64: 100n TMAG B12, Capacitor_SMD:C_0402_1005Metric, symbol Device:C
- removed C65: 100n TMAG B13, Capacitor_SMD:C_0402_1005Metric, symbol Device:C
- removed C66: 100n TMAG B14, Capacitor_SMD:C_0402_1005Metric, symbol Device:C
- removed C67: 100n TMAG B15, Capacitor_SMD:C_0402_1005Metric, symbol Device:C
- removed C68: 100n TMAG B16, Capacitor_SMD:C_0402_1005Metric, symbol Device:C
- removed C69: 100n TMAG B17, Capacitor_SMD:C_0402_1005Metric, symbol Device:C
- removed C70: 100n TMAG B18, Capacitor_SMD:C_0402_1005Metric, symbol Device:C
- removed C71: 10u USB 5V IN, Capacitor_SMD:C_0402_1005Metric, symbol Device:C
- removed C72: 10u RX 3V3, Capacitor_SMD:C_0402_1005Metric, symbol Device:C
- removed D1, D21, D41: ESD441DPYR USB VBUS, Diode_SMD:D_0201_0603Metric, symbol kaboard_custom:ESD441DPYR_PASSIVE
- removed D10: WL-ICLED A08, kaboard_custom:U_Wurth_WL-ICLED_1312020030000, symbol kaboard_custom:WL_ICLED_1312020030000
- removed D11: WL-ICLED A09, kaboard_custom:U_Wurth_WL-ICLED_1312020030000, symbol kaboard_custom:WL_ICLED_1312020030000
- removed D12: WL-ICLED A10, kaboard_custom:U_Wurth_WL-ICLED_1312020030000, symbol kaboard_custom:WL_ICLED_1312020030000
- removed D13: WL-ICLED A11, kaboard_custom:U_Wurth_WL-ICLED_1312020030000, symbol kaboard_custom:WL_ICLED_1312020030000
- removed D14: WL-ICLED A12, kaboard_custom:U_Wurth_WL-ICLED_1312020030000, symbol kaboard_custom:WL_ICLED_1312020030000
- removed D15: WL-ICLED A13, kaboard_custom:U_Wurth_WL-ICLED_1312020030000, symbol kaboard_custom:WL_ICLED_1312020030000
- removed D16: WL-ICLED A14, kaboard_custom:U_Wurth_WL-ICLED_1312020030000, symbol kaboard_custom:WL_ICLED_1312020030000
- removed D17: WL-ICLED A15, kaboard_custom:U_Wurth_WL-ICLED_1312020030000, symbol kaboard_custom:WL_ICLED_1312020030000
- removed D18: WL-ICLED A16, kaboard_custom:U_Wurth_WL-ICLED_1312020030000, symbol kaboard_custom:WL_ICLED_1312020030000
- removed D19: WL-ICLED A17, kaboard_custom:U_Wurth_WL-ICLED_1312020030000, symbol kaboard_custom:WL_ICLED_1312020030000
- removed D2: LEFT STATUS LED, LED_SMD:LED_0603_1608Metric, symbol Device:LED
- removed D20: WL-ICLED A18, kaboard_custom:U_Wurth_WL-ICLED_1312020030000, symbol kaboard_custom:WL_ICLED_1312020030000
- removed D22: RIGHT STATUS LED, LED_SMD:LED_0603_1608Metric, symbol Device:LED
- removed D23: WL-ICLED B01, kaboard_custom:U_Wurth_WL-ICLED_1312020030000, symbol kaboard_custom:WL_ICLED_1312020030000
- removed D24: WL-ICLED B02, kaboard_custom:U_Wurth_WL-ICLED_1312020030000, symbol kaboard_custom:WL_ICLED_1312020030000
- removed D25: WL-ICLED B03, kaboard_custom:U_Wurth_WL-ICLED_1312020030000, symbol kaboard_custom:WL_ICLED_1312020030000
- removed D26: WL-ICLED B04, kaboard_custom:U_Wurth_WL-ICLED_1312020030000, symbol kaboard_custom:WL_ICLED_1312020030000
- removed D27: WL-ICLED B05, kaboard_custom:U_Wurth_WL-ICLED_1312020030000, symbol kaboard_custom:WL_ICLED_1312020030000
- removed D28: WL-ICLED B06, kaboard_custom:U_Wurth_WL-ICLED_1312020030000, symbol kaboard_custom:WL_ICLED_1312020030000
- removed D29: WL-ICLED B07, kaboard_custom:U_Wurth_WL-ICLED_1312020030000, symbol kaboard_custom:WL_ICLED_1312020030000
- removed D3: WL-ICLED A01, kaboard_custom:U_Wurth_WL-ICLED_1312020030000, symbol kaboard_custom:WL_ICLED_1312020030000
- removed D30: WL-ICLED B08, kaboard_custom:U_Wurth_WL-ICLED_1312020030000, symbol kaboard_custom:WL_ICLED_1312020030000
- removed D31: WL-ICLED B09, kaboard_custom:U_Wurth_WL-ICLED_1312020030000, symbol kaboard_custom:WL_ICLED_1312020030000
- removed D32: WL-ICLED B10, kaboard_custom:U_Wurth_WL-ICLED_1312020030000, symbol kaboard_custom:WL_ICLED_1312020030000
- removed D33: WL-ICLED B11, kaboard_custom:U_Wurth_WL-ICLED_1312020030000, symbol kaboard_custom:WL_ICLED_1312020030000
- removed D34: WL-ICLED B12, kaboard_custom:U_Wurth_WL-ICLED_1312020030000, symbol kaboard_custom:WL_ICLED_1312020030000
- removed D35: WL-ICLED B13, kaboard_custom:U_Wurth_WL-ICLED_1312020030000, symbol kaboard_custom:WL_ICLED_1312020030000
- removed D36: WL-ICLED B14, kaboard_custom:U_Wurth_WL-ICLED_1312020030000, symbol kaboard_custom:WL_ICLED_1312020030000
- removed D37: WL-ICLED B15, kaboard_custom:U_Wurth_WL-ICLED_1312020030000, symbol kaboard_custom:WL_ICLED_1312020030000
- removed D38: WL-ICLED B16, kaboard_custom:U_Wurth_WL-ICLED_1312020030000, symbol kaboard_custom:WL_ICLED_1312020030000
- removed D39: WL-ICLED B17, kaboard_custom:U_Wurth_WL-ICLED_1312020030000, symbol kaboard_custom:WL_ICLED_1312020030000
- removed D4: WL-ICLED A02, kaboard_custom:U_Wurth_WL-ICLED_1312020030000, symbol kaboard_custom:WL_ICLED_1312020030000
- removed D40: WL-ICLED B18, kaboard_custom:U_Wurth_WL-ICLED_1312020030000, symbol kaboard_custom:WL_ICLED_1312020030000
- removed D42: STATUS LED, LED_SMD:LED_0603_1608Metric, symbol Device:LED
- removed D5: WL-ICLED A03, kaboard_custom:U_Wurth_WL-ICLED_1312020030000, symbol kaboard_custom:WL_ICLED_1312020030000
- removed D6: WL-ICLED A04, kaboard_custom:U_Wurth_WL-ICLED_1312020030000, symbol kaboard_custom:WL_ICLED_1312020030000
- removed D7: WL-ICLED A05, kaboard_custom:U_Wurth_WL-ICLED_1312020030000, symbol kaboard_custom:WL_ICLED_1312020030000
- removed D8: WL-ICLED A06, kaboard_custom:U_Wurth_WL-ICLED_1312020030000, symbol kaboard_custom:WL_ICLED_1312020030000
- removed D9: WL-ICLED A07, kaboard_custom:U_Wurth_WL-ICLED_1312020030000, symbol kaboard_custom:WL_ICLED_1312020030000
- removed J1, J11, J6: USB_C_Receptacle_PowerOnly_6P, Connector_USB:USB_C_Receptacle_GCT_USB4125-xx-x-0190_6P_TopMnt_Horizontal, symbol Connector:USB_C_Receptacle_PowerOnly_6P
- removed J10, J5: nRF SWD, Connector_PinHeader_2.54mm:PinHeader_1x05_P2.54mm_Vertical, symbol Connector_Generic:Conn_01x05
- removed J12, J3, J8: SH1106 1.3in 4-wire OLED, Connector_PinHeader_2.54mm:PinHeader_1x04_P2.54mm_Vertical, symbol Connector_Generic:Conn_01x04
- removed J13: Receiver nRF SWD, Connector_PinHeader_2.54mm:PinHeader_1x05_P2.54mm_Vertical, symbol Connector_Generic:Conn_01x05
- removed J2, J7: AS584070 BATTERY / 10k NTC, Connector_JST:JST_PH_B3B-PH-K_1x03_P2.00mm_Vertical, symbol Connector:Conn_01x03_Pin
- removed J4, J9: STM32 SWD, Connector_PinHeader_2.54mm:PinHeader_1x05_P2.54mm_Vertical, symbol Connector_Generic:Conn_01x05
- removed L1, L3: 2.2uH TPS63031, Inductor_SMD:L_0603_1608Metric, symbol Device:L
- removed L2, L4: 1uH RGB BOOST, Inductor_SMD:L_0603_1608Metric, symbol Device:L
- removed L5, L6, L7: 10uH nRF DCDC, Inductor_SMD:L_0603_1608Metric, symbol Device:L
- removed R1, R15, R29: 5.1k USB CC1, Resistor_SMD:R_0402_1005Metric, symbol Device:R
- removed R10, R24: 330k BAT_SENSE bottom, Resistor_SMD:R_0402_1005Metric, symbol Device:R
- removed R11, R25: 330R RGB data, Resistor_SMD:R_0402_1005Metric, symbol Device:R
- removed R12, R26: 732k RGB FB top, Resistor_SMD:R_0402_1005Metric, symbol Device:R
- removed R13, R27: 100k RGB FB bottom, Resistor_SMD:R_0402_1005Metric, symbol Device:R
- removed R14, R28, R34: 1k STATUS LED, Resistor_SMD:R_0402_1005Metric, symbol Device:R
- removed R16, R2, R30: 5.1k USB CC2, Resistor_SMD:R_0402_1005Metric, symbol Device:R
- removed R17, R3: 18k BQ ILIM/VSET, Resistor_SMD:R_0402_1005Metric, symbol Device:R
- removed R18, R4: 845R BQ ISET, Resistor_SMD:R_0402_1005Metric, symbol Device:R
- removed R19, R31, R5: 10k nRF RESET pullup, Resistor_SMD:R_0402_1005Metric, symbol Device:R
- removed R20, R6: 10k BOOT0 pulldown, Resistor_SMD:R_0402_1005Metric, symbol Device:R
- removed R21, R32, R7: 4.7k I2C SDA pullup, Resistor_SMD:R_0402_1005Metric, symbol Device:R
- removed R22, R33, R8: 4.7k I2C SCL pullup, Resistor_SMD:R_0402_1005Metric, symbol Device:R
- removed R23, R9: 1M BAT_SENSE top, Resistor_SMD:R_0402_1005Metric, symbol Device:R
- removed U1, U27: STM32G431RBTx, Package_QFP:LQFP-64_10x10mm_P0.5mm, symbol MCU_ST_STM32G4:STM32G431RBTx
- removed U10: TMAG5253 A02, kaboard_custom:Kaboard_JadePro_TMAG5253, symbol kaboard_custom:TMAG5253BA3IQDMRR
- removed U11: TMAG5253 A03, kaboard_custom:Kaboard_JadePro_TMAG5253, symbol kaboard_custom:TMAG5253BA3IQDMRR
- removed U12: TMAG5253 A04, kaboard_custom:Kaboard_JadePro_TMAG5253, symbol kaboard_custom:TMAG5253BA3IQDMRR
- removed U13: TMAG5253 A05, kaboard_custom:Kaboard_JadePro_TMAG5253, symbol kaboard_custom:TMAG5253BA3IQDMRR
- removed U14: TMAG5253 A06, kaboard_custom:Kaboard_JadePro_TMAG5253, symbol kaboard_custom:TMAG5253BA3IQDMRR
- removed U15: TMAG5253 A07, kaboard_custom:Kaboard_JadePro_TMAG5253, symbol kaboard_custom:TMAG5253BA3IQDMRR
- removed U16: TMAG5253 A08, kaboard_custom:Kaboard_JadePro_TMAG5253, symbol kaboard_custom:TMAG5253BA3IQDMRR
- removed U17: TMAG5253 A09, kaboard_custom:Kaboard_JadePro_TMAG5253, symbol kaboard_custom:TMAG5253BA3IQDMRR
- removed U18: TMAG5253 A10, kaboard_custom:Kaboard_JadePro_TMAG5253, symbol kaboard_custom:TMAG5253BA3IQDMRR
- removed U19: TMAG5253 A11, kaboard_custom:Kaboard_JadePro_TMAG5253, symbol kaboard_custom:TMAG5253BA3IQDMRR
- removed U2, U28, U52: MDBT50Q-1MV2, RF_Module:Raytac_MDBT50Q, symbol RF_Module:MDBT50Q-1MV2
- removed U20: TMAG5253 A12, kaboard_custom:Kaboard_JadePro_TMAG5253, symbol kaboard_custom:TMAG5253BA3IQDMRR
- removed U21: TMAG5253 A13, kaboard_custom:Kaboard_JadePro_TMAG5253, symbol kaboard_custom:TMAG5253BA3IQDMRR
- removed U22: TMAG5253 A14, kaboard_custom:Kaboard_JadePro_TMAG5253, symbol kaboard_custom:TMAG5253BA3IQDMRR
- removed U23: TMAG5253 A15, kaboard_custom:Kaboard_JadePro_TMAG5253, symbol kaboard_custom:TMAG5253BA3IQDMRR
- removed U24: TMAG5253 A16, kaboard_custom:Kaboard_JadePro_TMAG5253, symbol kaboard_custom:TMAG5253BA3IQDMRR
- removed U25: TMAG5253 A17, kaboard_custom:Kaboard_JadePro_TMAG5253, symbol kaboard_custom:TMAG5253BA3IQDMRR
- removed U26: TMAG5253 A18, kaboard_custom:Kaboard_JadePro_TMAG5253, symbol kaboard_custom:TMAG5253BA3IQDMRR
- removed U29, U3: BQ25185DLHR, Package_DFN_QFN:Texas_DLH0010A_WSON-10-1EP_2.2x2mm_P0.4mm_EP0.9x1.5mm, symbol kaboard_custom:BQ25185DLHR
- removed U30, U4: TPS63031DSK, Package_SON:WSON-10-1EP_2.5x2.5mm_P0.5mm_EP1.2x2mm, symbol Regulator_Switching:TPS63031DSK
- removed U31, U5: TPS61022 RGB BOOST, Package_DFN_QFN:Texas_RWU0007A_VQFN-7_2x2mm_P0.5mm, symbol Converter_DCDC:TPS61022
- removed U32, U6: 74AHCT1G125, Package_TO_SOT_SMD:SOT-23-5, symbol 74xGxx:74AHCT1G125
- removed U33, U54, U7: TPS22919DCK, Package_TO_SOT_SMD:SOT-363_SC-70-6, symbol Power_Management:TPS22919DCK
- removed U34: TMAG5253 B01, kaboard_custom:Kaboard_JadePro_TMAG5253, symbol kaboard_custom:TMAG5253BA3IQDMRR
- removed U35: TMAG5253 B02, kaboard_custom:Kaboard_JadePro_TMAG5253, symbol kaboard_custom:TMAG5253BA3IQDMRR
- removed U36: TMAG5253 B03, kaboard_custom:Kaboard_JadePro_TMAG5253, symbol kaboard_custom:TMAG5253BA3IQDMRR
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Connections:
- no-connect marks 162 -> 0
Other:
- added sheet LEFT HALF (left.kicad_sch)
- added sheet RIGHT HALF (right-half.kicad_sch)
- added sheet USB RECEIVER (usb-receiver.kicad_sch)
- note added: "1S LiPo power • STM32 sensing • nRF52840 wireless • 18 Hall channels • RGB"
- note added: "Functional hierarchy for the complete wireless keyboard system"
- note added: "KABOARD V3 — UNIFIED HARDWARE"
- note added: "LEFT KEYBOARD HALF"
- note added: "Open each sheet for detailed functional circuitry. Net namespaces: L_ • R_ • RX_"
- note added: "RIGHT KEYBOARD HALF"
- note added: "USB RECEIVER"
- note added: "USB-C interface • nRF52840 radio/HID • optional display interface"
- note removed: "18× TMAG5253 — 3 ENABLE GROUPS / 18 ADC CHANNELS"
- note removed: "18× WL-ICLED — 5V SWITCHED RAIL / AHCT DATA LEVEL SHIFT"
- note removed: "DISPLAY: 4-WIRE SH1106 MODULE (VCC / GND / SCL / SDA)"
- note removed: "KABOARD V3 — ELECTRICAL SCHEMATIC"
- note removed: "LEFT HALF — INDEPENDENT 1S LiPo / WIRELESS"
- note removed: "L_* = LEFT HALF R_* = RIGHT HALF RX_* = USB RECEIVER"
- note removed: "OPTIONAL DISPLAY: 4-WIRE SH1106 MODULE"
- note removed: "POWER / CHARGE / 3V3 / 5V RGB"
- note removed: "RECEIVER — USB HID / nRF52840"
- note removed: "RIGHT HALF — INDEPENDENT 1S LiPo / WIRELESS"
- note removed: "STM32 ACQUISITION / CALIBRATION / ACTUATION"
- note removed: "SWD: STM32 + nRF52840"
- note removed: "SWD: nRF52840"
- note removed: "USB POWER / 3V3 / DISPLAY"
- note removed: "nRF52840 RADIO / BATTERY TELEMETRY / I²C"
