File: kaboardv3-hw/left.kicad_sch (KiCad schematic)
At the start: 85 parts, among them J1 USB-C 5V IN, J2 BATTERY + NTC, J3 SH1106 OLED, J4 STM32 SWD, J5 nRF SWD, U1 STM32G431RBTx, U10 TMAG5253 + RGB, U11 TMAG5253 + RGB, U12 TMAG5253 + RGB, U13 TMAG5253 + RGB, U14 TMAG5253 + RGB, U15 TMAG5253 + RGB, U16 TMAG5253 + RGB, U17 TMAG5253 + RGB, U18 TMAG5253 + RGB, U19 TMAG5253 + RGB, U2 MDBT50Q-1MV2, U20 TMAG5253 + RGB, U21 TMAG5253 + RGB, U22 TMAG5253 + RGB, U23 TMAG5253 + RGB, U24 TMAG5253 + RGB, U25 TMAG5253 + RGB, U26 TMAG5253 + RGB, U3 BQ25185DLHR, U4 TPS63031DSK, U5 TPS61022, U6 74AHCT1G125, U7 TPS22919DCK, U9 TMAG5253 + RGB, Y1 32.768kHz

Commit message: organize unified schematics
Connections:
- net L_LED_5V: no longer U5.4 (FB)
- net L_RGB_FB: now also U5.4 (FB)
Other:
- note added: "TPS61022 FB divider: 732k / 100k sets 5 V per TI reference design."
- note removed: "Review: FB is presently tied to VOUT; divider midpoint is separate."
