File: kaboardv3-hw/right-half.kicad_sch (KiCad schematic)
At the start: 85 parts, among them J1 USB-C 5V IN, J2 BATTERY + NTC, J3 SH1106 OLED, J4 STM32 SWD, J5 nRF SWD, U1 STM32G431RBTx, U10 TMAG5253 + RGB, U11 TMAG5253 + RGB, U12 TMAG5253 + RGB, U13 TMAG5253 + RGB, U14 TMAG5253 + RGB, U15 TMAG5253 + RGB, U16 TMAG5253 + RGB, U17 TMAG5253 + RGB, U18 TMAG5253 + RGB, U19 TMAG5253 + RGB, U2 MDBT50Q-1MV2, U20 TMAG5253 + RGB, U21 TMAG5253 + RGB, U22 TMAG5253 + RGB, U23 TMAG5253 + RGB, U24 TMAG5253 + RGB, U25 TMAG5253 + RGB, U26 TMAG5253 + RGB, U3 BQ25185DLHR, U4 TPS63031DSK, U5 TPS61022, U6 74AHCT1G125, U7 TPS22919DCK, U9 TMAG5253 + RGB, Y1 32.768kHz

Commit message: organize unified schematics
Parts:
- removed C1, C16, C3: 1u, Capacitor_SMD:C_0402_1005Metric, symbol Device:C
- removed C10, C15, C17, C18, C19, C20, C21, C22, C23, C24, C25, C26, C27, C28, C29, C30, C31, C32, C33, C34, C35, C6, C7, C8, C9: 100n, Capacitor_SMD:C_0402_1005Metric, symbol Device:C
- removed C11, C12: 12p, Capacitor_SMD:C_0402_1005Metric, symbol Device:C
- removed C13, C2, C4, C5: 10u, Capacitor_SMD:C_0402_1005Metric, symbol Device:C
- removed C14: 47u, Capacitor_SMD:C_0402_1005Metric, symbol Device:C
- removed D1: ESD441DPYR, Diode_SMD:D_0201_0603Metric, symbol kaboard_custom:ESD441DPYR_PASSIVE
- removed D2: STATUS, LED_SMD:LED_0603_1608Metric, symbol Device:LED
- removed J1: USB-C 5V IN, Connector_USB:USB_C_Receptacle_GCT_USB4125-xx-x-0190_6P_TopMnt_Horizontal, symbol Connector:USB_C_Receptacle_PowerOnly_6P
- removed J2: BATTERY + NTC, Connector_JST:JST_PH_B3B-PH-K_1x03_P2.00mm_Vertical, symbol Connector:Conn_01x03_Pin
- removed J3: SH1106 OLED, Connector_PinHeader_2.54mm:PinHeader_1x04_P2.54mm_Vertical, symbol Connector_Generic:Conn_01x04
- removed J4: STM32 SWD, Connector_PinHeader_2.54mm:PinHeader_1x05_P2.54mm_Vertical, symbol Connector_Generic:Conn_01x05
- removed J5: nRF SWD, Connector_PinHeader_2.54mm:PinHeader_1x05_P2.54mm_Vertical, symbol Connector_Generic:Conn_01x05
- removed L1: 2.2uH, Inductor_SMD:L_0603_1608Metric, symbol Device:L
- removed L2: 1uH, Inductor_SMD:L_0603_1608Metric, symbol Device:L
- removed L6: 10uH, Inductor_SMD:L_0603_1608Metric, symbol Device:L
- removed R1: 5.1k, Resistor_SMD:R_0402_1005Metric, symbol Device:R_Small
- removed R10: 330k, Resistor_SMD:R_0402_1005Metric, symbol Device:R
- removed R11: 330R, Resistor_SMD:R_0402_1005Metric, symbol Device:R
- removed R12: 732k, Resistor_SMD:R_0402_1005Metric, symbol Device:R
- removed R13: 100k, Resistor_SMD:R_0402_1005Metric, symbol Device:R
- removed R14: 1k, Resistor_SMD:R_0402_1005Metric, symbol Device:R
- removed R2: 5.1k, Resistor_SMD:R_0402_1005Metric, symbol Device:R
- removed R3: 18k, Resistor_SMD:R_0402_1005Metric, symbol Device:R
- removed R4: 845R, Resistor_SMD:R_0402_1005Metric, symbol Device:R
- removed R5, R6: 10k, Resistor_SMD:R_0402_1005Metric, symbol Device:R
- removed R7, R8: 4.7k, Resistor_SMD:R_0402_1005Metric, symbol Device:R
- removed R9: 1M, Resistor_SMD:R_0402_1005Metric, symbol Device:R
- removed U1: STM32G431RBTx, Package_QFP:LQFP-64_10x10mm_P0.5mm, symbol MCU_ST_STM32G4:STM32G431RBTx
- removed U10, U11, U12, U13, U14, U15, U16, U17, U18, U19, U20, U21, U22, U23, U24, U25, U26, U9: TMAG5253 + RGB, kaboard_custom:Kaboard_JadePro_TMAG5253_RGB_Sides, symbol kaboard_custom:Kaboard_JadePro_TMAG5253_RGB
- removed U2: MDBT50Q-1MV2, RF_Module:Raytac_MDBT50Q, symbol RF_Module:MDBT50Q-1MV2
- removed U3: BQ25185DLHR, Package_DFN_QFN:Texas_DLH0010A_WSON-10-1EP_2.2x2mm_P0.4mm_EP0.9x1.5mm, symbol kaboard_custom:BQ25185DLHR
- removed U4: TPS63031DSK, Package_SON:WSON-10-1EP_2.5x2.5mm_P0.5mm_EP1.2x2mm, symbol Regulator_Switching:TPS63031DSK
- removed U5: TPS61022, Package_DFN_QFN:Texas_RWU0007A_VQFN-7_2x2mm_P0.5mm, symbol Converter_DCDC:TPS61022
- removed U6: 74AHCT1G125, Package_TO_SOT_SMD:SOT-23-5, symbol 74xGxx:74AHCT1G125
- removed U7: TPS22919DCK, Package_TO_SOT_SMD:SOT-363_SC-70-6, symbol Power_Management:TPS22919DCK
- removed Y1: 32.768kHz, Crystal:Crystal_SMD_3215-2Pin_3.2x1.5mm, symbol Device:Crystal
- added C36, C38, C51: 1u, Capacitor_SMD:C_0402_1005Metric, symbol Device:C
- added C37, C39, C40, C48: 10u, Capacitor_SMD:C_0402_1005Metric, symbol Device:C
- added C41, C42, C43, C44, C45, C50, C52, C53, C54, C55, C56, C57, C58, C59, C60, C61, C62, C63, C64, C65, C66, C67, C68, C69, C70: 100n, Capacitor_SMD:C_0402_1005Metric, symbol Device:C
- added C46, C47: 12p, Capacitor_SMD:C_0402_1005Metric, symbol Device:C
- added C49: 47u, Capacitor_SMD:C_0402_1005Metric, symbol Device:C
- added D3: ESD441DPYR, Diode_SMD:D_0201_0603Metric, symbol kaboard_custom:ESD441DPYR_PASSIVE
- added D4: STATUS, LED_SMD:LED_0603_1608Metric, symbol Device:LED
- added J10: nRF SWD, Connector_PinHeader_2.54mm:PinHeader_1x05_P2.54mm_Vertical, symbol Connector_Generic:Conn_01x05
- added J6: USB-C 5V IN, Connector_USB:USB_C_Receptacle_GCT_USB4125-xx-x-0190_6P_TopMnt_Horizontal, symbol Connector:USB_C_Receptacle_PowerOnly_6P
- added J7: BATTERY + NTC, Connector_JST:JST_PH_B3B-PH-K_1x03_P2.00mm_Vertical, symbol Connector:Conn_01x03_Pin
- added J8: SH1106 OLED, Connector_PinHeader_2.54mm:PinHeader_1x04_P2.54mm_Vertical, symbol Connector_Generic:Conn_01x04
- added J9: STM32 SWD, Connector_PinHeader_2.54mm:PinHeader_1x05_P2.54mm_Vertical, symbol Connector_Generic:Conn_01x05
- added L3: 2.2uH, Inductor_SMD:L_0603_1608Metric, symbol Device:L
- added L4: 1uH, Inductor_SMD:L_0603_1608Metric, symbol Device:L
- added L7: 10uH, Inductor_SMD:L_0603_1608Metric, symbol Device:L
- added R15: 5.1k, Resistor_SMD:R_0402_1005Metric, symbol Device:R_Small
- added R16: 5.1k, Resistor_SMD:R_0402_1005Metric, symbol Device:R
- added R17: 18k, Resistor_SMD:R_0402_1005Metric, symbol Device:R
- added R18: 845R, Resistor_SMD:R_0402_1005Metric, symbol Device:R
- added R19, R20: 10k, Resistor_SMD:R_0402_1005Metric, symbol Device:R
- added R21, R22: 4.7k, Resistor_SMD:R_0402_1005Metric, symbol Device:R
- added R23: 1M, Resistor_SMD:R_0402_1005Metric, symbol Device:R
- added R24: 330k, Resistor_SMD:R_0402_1005Metric, symbol Device:R
- added R25: 330R, Resistor_SMD:R_0402_1005Metric, symbol Device:R
- added R26: 732k, Resistor_SMD:R_0402_1005Metric, symbol Device:R
- added R27: 100k, Resistor_SMD:R_0402_1005Metric, symbol Device:R
- added R28: 1k, Resistor_SMD:R_0402_1005Metric, symbol Device:R
- added U27: STM32G431RBTx, Package_QFP:LQFP-64_10x10mm_P0.5mm, symbol MCU_ST_STM32G4:STM32G431RBTx
- added U28: MDBT50Q-1MV2, RF_Module:Raytac_MDBT50Q, symbol RF_Module:MDBT50Q-1MV2
- added U29: BQ25185DLHR, Package_DFN_QFN:Texas_DLH0010A_WSON-10-1EP_2.2x2mm_P0.4mm_EP0.9x1.5mm, symbol kaboard_custom:BQ25185DLHR
- added U30: TPS63031DSK, Package_SON:WSON-10-1EP_2.5x2.5mm_P0.5mm_EP1.2x2mm, symbol Regulator_Switching:TPS63031DSK
- added U31: TPS61022, Package_DFN_QFN:Texas_RWU0007A_VQFN-7_2x2mm_P0.5mm, symbol Converter_DCDC:TPS61022
- added U32: 74AHCT1G125, Package_TO_SOT_SMD:SOT-23-5, symbol 74xGxx:74AHCT1G125
- added U33: TPS22919DCK, Package_TO_SOT_SMD:SOT-363_SC-70-6, symbol Power_Management:TPS22919DCK
- added U34, U35, U36, U37, U38, U39, U40, U41, U42, U43, U44, U45, U46, U47, U48, U49, U50, U51: TMAG5253 + RGB, kaboard_custom:Kaboard_JadePro_TMAG5253_RGB_Sides, symbol kaboard_custom:Kaboard_JadePro_TMAG5253_RGB
- added Y2: 32.768kHz, Crystal:Crystal_SMD_3215-2Pin_3.2x1.5mm, symbol Device:Crystal
Connections:
- new net R_3V3: C40.1, C41.1, C42.1, C43.1, C44.1, C45.1, C48.1, C53.1, C54.1, C55.1, C56.1, C57.1, C58.1, C59.1, C60.1, C61.1, C62.1, C63.1, C64.1, C65.1, C66.1, C67.1, C68.1, C69.1, C70.1, J10.1 (Pin_1), J9.1 (Pin_1), L4.1, L7.2, R19.2, R21.1, R22.1, U27.1 (VBAT), U27.16 (VDD), U27.28 (VREF+), U27.29 (VDDA), U27.32 (VDD), U27.48 (VDD), U27.64 (VDD), U28.28 (VDD), U28.30 (VDDH), U28.32 (VBUS), U30.1 (VOUT), U30.10 (FB), U31.7 (VIN), U33.1 (IN), U34.1 (VCC), U35.1 (VCC), U36.1 (VCC), U37.1 (VCC), U38.1 (VCC), U39.1 (VCC), U40.1 (VCC), U41.1 (VCC), U42.1 (VCC), U43.1 (VCC), U44.1 (VCC), U45.1 (VCC), U46.1 (VCC), U47.1 (VCC), U48.1 (VCC), U49.1 (VCC), U50.1 (VCC), U51.1 (VCC)
- new net R_BAT: C38.1, J7.1 (Pin_1), R23.1, U29.2 (BAT)
- new net R_BAT_SENSE: R23.2, R24.1, U28.10 (P0.29)
- new net R_BOOT0: R20.1, U27.61 (PB8)
- new net R_BQ_ILIM: R17.1, U29.7 (ILIM/VSET)
- new net R_BQ_ISET: R18.1, U29.8 (ISET)
- new net R_DISPLAY_EN: U28.49 (P0.25), U33.3 (ON)
- new net R_DISPLAY_SCL: J8.3 (Pin_3), R22.2, U28.19 (P0.26)
- new net R_DISPLAY_SDA: J8.4 (Pin_4), R21.2, U28.16 (P0.27)
- new net R_GND: C36.2, C37.2, C38.2, C39.2, C40.2, C41.2, C42.2, C43.2, C44.2, C45.2, C46.2, C47.2, C48.2, C49.2, C50.2, C51.2, C52.2, C53.2, C54.2, C55.2, C56.2, C57.2, C58.2, C59.2, C60.2, C61.2, C62.2, C63.2, C64.2, C65.2, C66.2, C67.2, C68.2, C69.2, C70.2, D3.2 (GND), D4.1 (K), J10.2 (Pin_2), J6.A12 (GND), J6.B12 (GND), J6.SH (SHIELD), J7.3 (Pin_3), J8.2 (Pin_2), J9.2 (Pin_2), R15.2, R16.2, R17.2, R18.2, R20.2, R24.2, R27.2, U27.15 (VSS), U27.27 (VSSA), U27.31 (VSS), U27.47 (VSS), U27.63 (VSS), U28.1 (GND), U28.15 (GND), U28.2 (GND), U28.33 (GND), U28.55 (GND), U29.11 (EP), U29.4 (/CE), U29.5 (GND), U30.11 (PGND), U30.3 (PGND), U30.7 (PS/SYNC), U30.9 (GND), U31.1 (GND), U31.6 (MODE), U32.1, U32.3 (GND), U33.2 (GND), U34.2 (GND), U34.5 (EP), U34.9 (LED_GND), U35.2 (GND), U35.5 (EP), U35.9 (LED_GND), U36.2 (GND), U36.5 (EP), U36.9 (LED_GND), U37.2 (GND), U37.5 (EP), U37.9 (LED_GND), U38.2 (GND), U38.5 (EP), U38.9 (LED_GND), U39.2 (GND), U39.5 (EP), U39.9 (LED_GND), U40.2 (GND), U40.5 (EP), U40.9 (LED_GND), U41.2 (GND), U41.5 (EP), U41.9 (LED_GND), U42.2 (GND), U42.5 (EP), U42.9 (LED_GND), U43.2 (GND), U43.5 (EP), U43.9 (LED_GND), U44.2 (GND), U44.5 (EP), U44.9 (LED_GND), U45.2 (GND), U45.5 (EP), U45.9 (LED_GND), U46.2 (GND), U46.5 (EP), U46.9 (LED_GND), U47.2 (GND), U47.5 (EP), U47.9 (LED_GND), U48.2 (GND), U48.5 (EP), U48.9 (LED_GND), U49.2 (GND), U49.5 (EP), U49.9 (LED_GND), U50.2 (GND), U50.5 (EP), U50.9 (LED_GND), U51.2 (GND), U51.5 (EP), U51.9 (LED_GND)
- new net R_HALL_EN_A: U27.38 (PC6), U34.3 (EN), U35.3 (EN), U36.3 (EN), U37.3 (EN), U38.3 (EN), U39.3 (EN)
- new net R_HALL_EN_B: U27.39 (PC7), U40.3 (EN), U41.3 (EN), U42.3 (EN), U43.3 (EN), U44.3 (EN), U45.3 (EN)
- new net R_HALL_EN_C: U27.40 (PC8), U46.3 (EN), U47.3 (EN), U48.3 (EN), U49.3 (EN), U50.3 (EN), U51.3 (EN)
- new net R_HALL_OUT_01: U27.8 (PC0), U34.4 (OUT)
- new net R_HALL_OUT_02: U27.9 (PC1), U35.4 (OUT)
- new net R_HALL_OUT_03: U27.10 (PC2), U36.4 (OUT)
- new net R_HALL_OUT_04: U27.11 (PC3), U37.4 (OUT)
- new net R_HALL_OUT_05: U27.12 (PA0), U38.4 (OUT)
- new net R_HALL_OUT_06: U27.13 (PA1), U39.4 (OUT)
- new net R_HALL_OUT_07: U27.14 (PA2), U40.4 (OUT)
- new net R_HALL_OUT_08: U27.17 (PA3), U41.4 (OUT)
- new net R_HALL_OUT_09: U27.18 (PA4), U42.4 (OUT)
- new net R_HALL_OUT_10: U27.19 (PA5), U43.4 (OUT)
- new net R_HALL_OUT_11: U27.20 (PA6), U44.4 (OUT)
- new net R_HALL_OUT_12: U27.21 (PA7), U45.4 (OUT)
- new net R_HALL_OUT_13: U27.22 (PC4), U46.4 (OUT)
- new net R_HALL_OUT_14: U27.23 (PC5), U47.4 (OUT)
- new net R_HALL_OUT_15: U27.24 (PB0), U48.4 (OUT)
- new net R_HALL_OUT_16: U27.25 (PB1), U49.4 (OUT)
- new net R_HALL_OUT_17: U27.26 (PB2), U50.4 (OUT)
- new net R_HALL_OUT_18: U27.33 (PB11), U51.4 (OUT)
- new net R_LED_5V: C49.1, C50.1, R26.1, U31.3 (VOUT), U32.5 (VCC), U34.6 (LED_VDD), U35.6 (LED_VDD), U36.6 (LED_VDD), U37.6 (LED_VDD), U38.6 (LED_VDD), U39.6 (LED_VDD), U40.6 (LED_VDD), U41.6 (LED_VDD), U42.6 (LED_VDD), U43.6 (LED_VDD), U44.6 (LED_VDD), U45.6 (LED_VDD), U46.6 (LED_VDD), U47.6 (LED_VDD), U48.6 (LED_VDD), U49.6 (LED_VDD), U50.6 (LED_VDD), U51.6 (LED_VDD)
- new net R_NRF_DCCH: L7.1, U28.31 (DCCH)
- new net R_NRF_RESET_N: J10.5 (Pin_5), R19.1, U28.40 (P0.18)
- new net R_NRF_XL1: C46.1, U28.17 (P0.00), Y2.1
- new net R_NRF_XL2: C47.1, U28.18 (P0.01), Y2.2
- new net R_NTC: J7.2 (Pin_2), U29.6 (TS/MR)
- new net R_OLED_VCC: C51.1, C52.1, J8.1 (Pin_1), U33.6 (OUT)
- new net R_RGB_CHAIN_01: U34.8 (LED_DOUT), U35.7 (LED_DIN)
- new net R_RGB_CHAIN_02: U35.8 (LED_DOUT), U36.7 (LED_DIN)
- new net R_RGB_CHAIN_03: U36.8 (LED_DOUT), U37.7 (LED_DIN)
- new net R_RGB_CHAIN_04: U37.8 (LED_DOUT), U38.7 (LED_DIN)
- new net R_RGB_CHAIN_05: U38.8 (LED_DOUT), U39.7 (LED_DIN)
- new net R_RGB_CHAIN_08: U40.8 (LED_DOUT), U41.7 (LED_DIN)
- new net R_RGB_CHAIN_09: U41.8 (LED_DOUT), U42.7 (LED_DIN)
- new net R_RGB_CHAIN_10: U42.8 (LED_DOUT), U43.7 (LED_DIN)
- new net R_RGB_CHAIN_11: U43.8 (LED_DOUT), U44.7 (LED_DIN)
- new net R_RGB_CHAIN_12: U44.8 (LED_DOUT), U45.7 (LED_DIN)
- new net R_RGB_CHAIN_14: U46.8 (LED_DOUT), U47.7 (LED_DIN)
- new net R_RGB_CHAIN_15: U47.8 (LED_DOUT), U48.7 (LED_DIN)
- new net R_RGB_CHAIN_16: U48.8 (LED_DOUT), U49.7 (LED_DIN)
- new net R_RGB_CHAIN_17: U49.8 (LED_DOUT), U50.7 (LED_DIN)
- new net R_RGB_CHAIN_18: U50.8 (LED_DOUT), U51.7 (LED_DIN)
- new net R_RGB_DATA_3V3: U27.42 (PA8), U32.2
- new net R_RGB_DATA_5V: R25.1, U32.4
- new net R_RGB_DIN_01: R25.2, U34.7 (LED_DIN)
- new net R_RGB_DIN_07: U39.8 (LED_DOUT), U40.7 (LED_DIN)
- new net R_RGB_DIN_13: U45.8 (LED_DOUT), U46.7 (LED_DIN)
- new net R_RGB_FB: R26.2, R27.1, U31.4 (FB)
- new net R_RGB_PWR_EN: U27.43 (PA9), U31.5 (EN)
- new net R_RGB_SW: L4.2, U31.2 (SW)
- new net R_SPI_CS_N: U27.51 (PA15), U28.44 (P0.20)
- new net R_SPI_MISO: U27.53 (PC11), U28.46 (P0.22)
- new net R_SPI_MOSI: U27.54 (PC12), U28.43 (P0.21)
- new net R_SPI_SCK: U27.52 (PC10), U28.42 (P0.19)
- new net R_STATUS_LED: R28.1, U28.48 (P0.24)
- new net R_STATUS_LED_A: D4.2 (A), R28.2
- new net R_STM_DATA_READY: U27.30 (PB10), U28.36 (P0.14)
- new net R_STM_RESET_N: J9.5 (Pin_5), U27.7 (PG10)
- new net R_STM_WAKE_NRF: U27.41 (PC9), U28.37 (P0.13)
- new net R_SWCLK_NRF: J10.4 (Pin_4), U28.53 (SWDCLK)
- new net R_SWCLK_STM: J9.4 (Pin_4), U27.50 (PA14)
- new net R_SWDIO_NRF: J10.3 (Pin_3), U28.51 (SWDIO)
- new net R_SWDIO_STM: J9.3 (Pin_3), U27.49 (PA13)
- new net R_SYS: C37.1, C39.1, U29.1 (SYS), U30.5 (VIN), U30.6 (EN), U30.8 (VINA)
- new net R_TPS_L1: L3.1, U30.4 (L1)
- new net R_TPS_L2: L3.2, U30.2 (L2)
- new net R_USB_CC1: J6.A5 (CC1), R15.1
- new net R_USB_CC2: J6.B5 (CC2), R16.1
- new net R_USB_VBUS: C36.1, D3.1 (IO), J6.A9 (VBUS), J6.B9 (VBUS), U29.10 (IN)
Other:
- note added: "KABOARD V3 / RIGHT HALF"
- note added: "RIGHT HALF | 18 Hall channels | 18 addressable key LEDs | STM32G431 + nRF52840 | USB-C charging"
- note added: "TPS61022 FB divider: 732k / 100k sets 5 V per TI reference design."
- note removed: "KABOARD V3 / LEFT HALF"
- note removed: "LEFT HALF | 18 Hall channels | 18 addressable key LEDs | STM32G431 + nRF52840 | USB-C charging"
- note removed: "Review: FB is presently tied to VOUT; divider midpoint is separate."
