File: receiver/kaboard-receiver.kicad_sch (KiCad schematic)
At the start: 25 parts, among them J11 USB_C_Receptacle_PowerOnly_6P, J12 SH1106 1.3in 4-wire OLED, J13 Receiver nRF SWD, U52 MDBT50Q-1MV2, U53 AP2112K-3.3, U54 TPS22919DCK, Y3 32.768kHz

Commit message: organize unified schematics
Connections:
- no-connect marks 44 -> 90
Other:
- note added: "32 kHz CLOCK + SWD"
- note added: "DISPLAY POWER + I2C"
- note added: "KABOARD V3 — RECEIVER / USB HID"
- note added: "STATUS INDICATOR"
- note added: "USB INPUT / PROTECTION / 3V3 POWER"
- note added: "nRF52840 RADIO / LOCAL SUPPORT"
- note removed: "18× TMAG5253 — 3 ENABLE GROUPS / 18 ADC CHANNELS"
- note removed: "18× WL-ICLED — 5V SWITCHED RAIL / AHCT DATA LEVEL SHIFT"
- note removed: "DISPLAY: 4-WIRE SH1106 MODULE (VCC / GND / SCL / SDA)"
- note removed: "KABOARD V3 — ELECTRICAL SCHEMATIC"
- note removed: "LEFT HALF — INDEPENDENT 1S LiPo / WIRELESS"
- note removed: "L_* = LEFT HALF R_* = RIGHT HALF RX_* = USB RECEIVER"
- note removed: "OPTIONAL DISPLAY: 4-WIRE SH1106 MODULE"
- note removed: "POWER / CHARGE / 3V3 / 5V RGB"
- note removed: "RECEIVER — USB HID / nRF52840"
- note removed: "RIGHT HALF — INDEPENDENT 1S LiPo / WIRELESS"
- note removed: "STM32 ACQUISITION / CALIBRATION / ACTUATION"
- note removed: "SWD: STM32 + nRF52840"
- note removed: "SWD: nRF52840"
- note removed: "USB POWER / 3V3 / DISPLAY"
- note removed: "nRF52840 RADIO / BATTERY TELEMETRY / I²C"
- moved on the sheet: C71, C72, C73, C74, C75, C76, C77, C78, C79, D41, D42, J11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
