File: right/kaboard-right.kicad_sch (KiCad schematic)
At the start: 85 parts, among them J10 nRF SWD, J6 USB_C_Receptacle_PowerOnly_6P, J7 AS584070 BATTERY / 10k NTC, J8 SH1106 1.3in 4-wire OLED, J9 STM32 SWD, U27 STM32G431RBTx, U28 MDBT50Q-1MV2, U29 BQ25185DLHR, U30 TPS63031DSK, U31 TPS61022 RGB BOOST, U32 74AHCT1G125, U33 TPS22919DCK, U34 Kaboard Jade Pro TMAG5253 + W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, U35 Kaboard Jade Pro TMAG5253 + W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, U36 Kaboard Jade Pro TMAG5253 + W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, U37 Kaboard Jade Pro TMAG5253 + W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, U38 Kaboard Jade Pro TMAG5253 + W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, U39 Kaboard Jade Pro TMAG5253 + W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, U40 Kaboard Jade Pro TMAG5253 + W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, U41 Kaboard Jade Pro TMAG5253 + W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, U42 Kaboard Jade Pro TMAG5253 + W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, U43 Kaboard Jade Pro TMAG5253 + W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, U44 Kaboard Jade Pro TMAG5253 + W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, U45 Kaboard Jade Pro TMAG5253 + W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, U46 Kaboard Jade Pro TMAG5253 + W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, U47 Kaboard Jade Pro TMAG5253 + W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, U48 Kaboard Jade Pro TMAG5253 + W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, U49 Kaboard Jade Pro TMAG5253 + W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, U50 Kaboard Jade Pro TMAG5253 + W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, U51 Kaboard Jade Pro TMAG5253 + W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, Y2 32.768kHz

Commit message: organize unified schematics
Parts:
- R15, R16, R17: footprint (none) -> Resistor_SMD:R_0402_1005Metric
Other:
- note added: "DEBUG — STM32 + nRF SWD"
- note added: "DISPLAY — SH1106 I2C"
- note added: "HALL SENSORS — 3 ENABLE GROUPS / 18 ADC"
- note added: "RIGHT BOARD — 1S LiPo / WIRELESS"
- note added: "STM32 — ACQUISITION / CALIBRATION / ACTUATION"
- note added: "USB / CHARGE / POWER"
- note added: "WL-ICLED — 5V RAIL / LEVEL SHIFT"
- note added: "nRF52840 — RADIO / BATTERY / I2C"
- note removed: "18× TMAG5253 — 3 ENABLE GROUPS / 18 ADC CHANNELS"
- note removed: "18× WL-ICLED — 5V SWITCHED RAIL / AHCT DATA LEVEL SHIFT"
- note removed: "DISPLAY: 4-WIRE SH1106 MODULE (VCC / GND / SCL / SDA)"
- note removed: "KABOARD V3 — ELECTRICAL SCHEMATIC"
- note removed: "LEFT HALF — INDEPENDENT 1S LiPo / WIRELESS"
- note removed: "L_* = LEFT HALF R_* = RIGHT HALF RX_* = USB RECEIVER"
- note removed: "OPTIONAL DISPLAY: 4-WIRE SH1106 MODULE"
- note removed: "POWER / CHARGE / 3V3 / 5V RGB"
- note removed: "RECEIVER — USB HID / nRF52840"
- note removed: "RIGHT HALF — INDEPENDENT 1S LiPo / WIRELESS"
- note removed: "STM32 ACQUISITION / CALIBRATION / ACTUATION"
- note removed: "SWD: STM32 + nRF52840"
- note removed: "SWD: nRF52840"
- note removed: "USB POWER / 3V3 / DISPLAY"
- note removed: "nRF52840 RADIO / BATTERY TELEMETRY / I²C"
- moved on the sheet: C36, C37, C38, C39, C40, C41, C42, C43, C44, C45, C48, C49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
